File: pcbs/left_pcbv2.kicad_pcb (KiCad board)
At the start: 2 copper layers, 156.2 x 81.9 mm, 77 parts

Commit message: fixed the bodge
Connections:
- S21 pad 1: P5 -> P4
- S43 pad 1: P5 -> P4
Routing:
- net P4: track 157.1 -> 219.3 mm
- net P5: track 206.5 -> 163.6 mm
Changed lines of the file:
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@@
 			(drillshape 0)
 			(scaleselection 1)
-			(outputdirectory "leftsidev2")
+			(outputdirectory "leftsidev2withSS")
 		)
 	)
@@
 			(size 2.6 2.6)
 			(layers "B.Cu" "B.Mask" "B.Paste")
-			(net 12 "P5")
+			(net 10 "P4")
 		)
 		(pad "2" smd rect
@@
 			(size 2.55 2.5)
 			(layers "B.Cu" "B.Mask" "B.Paste")
-			(net 12 "P5")
+			(net 10 "P4")
 		)
 		(pad "2" smd rect
@@
 	)
 	(segment
+		(start 207.285 160.545108)
+		(end 205.640892 158.901)
+		(width 0.2)
+		(layer "B.Cu")
+		(net 10)
+	)
+	(segment
 		(start 205.190892 136.101)
 		(end 201.882923 136.101)
@@
 	)
 	(segment
+		(start 202.899 135.016709)
+		(end 203.983291 136.101)
+		(width 0.2)
+		(layer "B.Cu")
+		(net 10)
+	)
+	(segment
 		(start 192.5 94.399)
 		(end 189.733291 94.399)
@@
 	)
 	(segment
+		(start 201.215961 157.784039)
+		(end 209.626 149.374)
+		(width 0.2)
+		(layer "B.Cu")
+		(net 10)
+	)
+	(segment
 		(start 192.5 94.399)
 		(end 195.149 91.75)
@@
 	)
 	(segment
+		(start 202.899 133.483291)
+		(end 202.899 135.016709)
+		(width 0.2)
+		(layer "B.Cu")
+		(net 10)
+	)
+	(segment
+		(start 200.132923 156.701)
+		(end 198.776 156.701)
+		(width 0.2)
+		(layer "B.Cu")
+		(net 10)
+	)
+	(segment
 		(start 187.75 98.101)
 		(end 187.632923 98.101)
@@
 	)
 	(segment
+		(start 205.640892 158.901)
+		(end 204.433291 158.901)
+		(width 0.2)
+		(layer "B.Cu")
+		(net 10)
+	)
+	(segment
 		(start 199.876 113.399)
 		(end 194.483291 113.399)
@@
 	)
 	(segment
+		(start 202.332923 158.901)
+		(end 201.215961 157.784039)
+		(width 0.2)
+		(layer "B.Cu")
+		(net 10)
+	)
+	(segment
+		(start 205.640892 158.901)
+		(end 202.332923 158.901)
+		(width 0.2)
+		(layer "B.Cu")
+		(net 10)
+	)
+	(segment
+		(start 201.215961 157.784039)
+		(end 200.132923 156.701)
+		(width 0.2)
+		(layer "B.Cu")
+		(net 10)
+	)
+	(segment
+		(start 205.516709 136.101)
+		(end 206.835 137.419291)
+		(width 0.2)
+		(layer "B.Cu")
+		(net 10)
+	)
+	(segment
 		(start 206.835 140.54)
 		(end 206.835 137.745108)
@@
 	)
 	(segment
+		(start 198.776 156.701)
+		(end 196.925 154.85)
+		(width 0.2)
+		(layer "B.Cu")
+		(net 10)
+	)
+	(segment
 		(start 220.75 91.75)
 		(end 220.75 103.99)
@@
 	)
 	(segment
+		(start 209.626 149.374)
+		(end 209.626 132.649)
+		(width 0.2)
+		(layer "B.Cu")
+		(net 10)
+	)
+	(segment
 		(start 200.126 113.649)
 		(end 199.876 113.399)
@@
 	)
 	(segment
+		(start 209.376 132.399)
+		(end 203.983291 132.399)
+		(width 0.2)
+		(layer "B.Cu")
+		(net 10)
+	)
+	(segment
 		(start 195.376 94.649)
 		(end 195.126 94.399)
@@
 	)
 	(segment
+		(start 206.835 137.419291)
+		(end 206.835 140.54)
+		(width 0.2)
+		(layer "B.Cu")
+		(net 10)
+	)
+	(segment
 		(start 195.376 104.649)
 		(end 195.376 94.649)
@@
 	)
 	(segment
+		(start 207.285 163.34)
+		(end 207.285 160.545108)
+		(width 0.2)
+		(layer "B.Cu")
+		(net 10)
+	)
+	(segment
 		(start 199.682923 133.901)
 		(end 198.326 133.901)
@@
 	)
 	(segment
+		(start 203.983291 136.101)
+		(end 205.516709 136.101)
+		(width 0.2)
+		(layer "B.Cu")
+		(net 10)
+	)
+	(segment
 		(start 201.882923 136.101)
 		(end 199.682923 133.901)
@@
 	)
 	(segment
+		(start 203.983291 132.399)
+		(end 202.899 133.483291)
+		(width 0.2)
+		(layer "B.Cu")
+		(net 10)
+	)
+	(segment
 		(start 192.382923 115.499368)
 		(end 192.382923 117.101)
@@
 	)
 	(segment
+		(start 209.626 132.649)
+		(end 209.376 132.399)
+		(width 0.2)
+		(layer "B.Cu")
+		(net 10)
+	)
+	(segment
 		(start 187.15 108)
 		(end 186.081 106.931)
@@
 	)
 	(segment
-		(start 207.285 160.545108)
-		(end 205.640892 158.901)
-		(width 0.2)
-		(layer "B.Cu")
-		(net 12)
-	)
-	(segment
 		(start 218.75 113.399)
 		(end 213.483291 113.399)
@@
 	)
 	(segment
-		(start 203.349 157.816709)
-		(end 203.349 156.283291)
-		(width 0.2)
-		(layer "B.Cu")
-		(net 12)
-	)
-	(segment
 		(start 236.285 160.545108)
 		(end 234.640892 158.901)
@@
 	)
 	(segment
-		(start 200.132923 156.701)
-		(end 198.776 156.701)
-		(width 0.2)
-		(layer "B.Cu")
-		(net 12)
-	)
-	(segment
 		(start 224.589892 136.5)
 		(end 222.115709 136.5)
@@
 	)
 	(segment
-		(start 205.640892 158.901)
-		(end 204.433291 158.901)
-		(width 0.2)
-		(layer "B.Cu")
-		(net 12)
-	)
-	(segment
 		(start 211.585 99.745108)
 		(end 209.940892 98.101)
@@
 	)
 	(segment
-		(start 204.782291 154.85)
-		(end 225.925 154.85)
-		(width 0.2)
-		(layer "B.Cu")
-		(net 12)
-	)
-	(segment
-		(start 202.332923 158.901)
-		(end 200.132923 156.701)
-		(width 0.2)
-		(layer "B.Cu")
-		(net 12)
-	)
-	(segment
-		(start 205.640892 158.901)
-		(end 202.332923 158.901)
-		(width 0.2)
-		(layer "B.Cu")
-		(net 12)
-	)
-	(segment
 		(start 219.516709 133.901)
 		(end 217.326 133.901)
@@
 	)
 	(segment
-		(start 198.776 156.701)
-		(end 196.925 154.85)
-		(width 0.2)
-		(layer "B.Cu")
-		(net 12)
-	)
-	(segment
 		(start 214.376 104.649)
 		(end 214.376 94.649)
@@
 	)
 	(segment
-		(start 207.285 163.34)
-		(end 207.285 160.545108)
-		(width 0.2)
-		(layer "B.Cu")
-		(net 12)
-	)
-	(segment
 		(start 234.640892 158.901)
 		(end 231.332923 158.901)
@@
 		(width 0.2)
 		(layer "B.Cu")
-		(net 12)
-	)
-	(segment
-		(start 204.433291 158.901)
-		(end 203.349 157.816709)
-		(width 0.2)
-		(layer "B.Cu")
-		(net 12)
-	)
-	(segment
-		(start 203.349 156.283291)
-		(end 204.782291 154.85)
-		(width 0.2)
-		(layer "B.Cu")
